File: grove_qwiic_breadboard/grove_qwiic_breadboard.kicad_pcb (KiCad board)
At the start: 2 copper layers, 33 x 14 mm, 16 parts, among them U1 AP7333-33SAG

Commit message: grove-qwiic-bb-bridge
Parts:
- CH6: moved to B.Cu
- moved C2 5.16 mm to (74.7, 66.4)
- moved U1 5.16 mm to (69.7, 67.3), turned to 180 degrees
- moved C1 3.36 mm to (72.8, 68.8)
- moved CH6 2.95 mm to (69.9, 75.2), turned to -90 degrees
- moved R2 1.63 mm to (74.3, 75.7)
- moved R1 1.63 mm to (74.3, 74.2)
Routing:
- net VCC: track 46.8 -> 48.3 mm, vias 2 -> 3
- net +3V3: track 19.5 -> 18.6 mm
- net /SCL: track 20.4 -> 19.4 mm, vias 1 -> 2
- net /SDA: track 18.3 -> 18.5 mm, vias 1 -> 2
- net GND: vias 17 -> 9
Other:
- board text added: "74th-"
- board text added: "B048-"
- board text added: "BbBridge"
- board text added: "GroveQwiic"
- board text added: "v1.0.0"
- board text removed: "74th-B048-v1.0.0"
- board text removed: "Bb Bridge"
- board text removed: "Grove Qwiic"
