File: grove_qwiic_breadboard_bridge/grove_qwiic_breadboard_bridge.kicad_pcb (KiCad board)
At the start: 2 copper layers, 33 x 14 mm, 16 parts, among them U1 AP7333-33SAG

Commit message: grove_qwiic_bb_bridge/v1.0.0
Parts:
- CH1, CH2, CH3, CH5: moved to B.Cu
Routing:
- net GND: track 7.62 -> 17.9 mm, vias 9 -> 10

Commit message: grove_qwiic_bb_bridge/v1.0.1
Parts:
- removed JP1: Jumper_2_Open, 74th:PinOut_Pin_2
- moved CH3 1.27 mm to (100.3, 73.7)
Routing:
- net +3V3: track 18.5 -> 10.3 mm, vias 1 -> 0
- net VCC: track 48.0 -> 50.0 mm, vias 3 -> 5
- net Net-(JP2-B1): track 20.2 -> 21.7 mm
- net Net-(CH3-Pad2): track 20.7 -> 22.1 mm
- net GND: vias 10 -> 11
Other:
- board size 33 x 14 mm -> 34.3 x 14 mm
- board text added: "v1.0.1"
- board text removed: "Vin=3V3"
- board text removed: "v1.0.0"
