File: grove_qwiic_breadboard_bridge/grove_qwiic_breadboard_bridge.kicad_sch (KiCad schematic)
At the start: 14 parts, among them U1 AP7333-33SAG

Commit message: grove_qwiic_bb_bridge/v1.0.0
Other:
- note added: "Breadboard Interface"
- note added: "Grove Socket"
- note added: "I2C Pullup"
- note added: "Qwiic Socket"
- note added: "SDA/SCL Select"
- company: (none) -> Atsushi Morimoto (@74th)
- title: (none) -> Grove Qwiic Breadboard Bridge
- moved on the sheet: C1, C2, C3, CH1, CH2, CH3, CH4, CH5, CH6, JP1, JP2, R1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

Commit message: grove_qwiic_bb_bridge/v1.0.1
Parts:
- removed JP1: Jumper_2_Open, 74th:PinOut_Pin_2, symbol 74th_Interface:Jumper_2
Other:
- moved on the sheet: C1, C2, U1
