File: test-lipo_battery/test-lipo_battery.kicad_pcb (KiCad board)
At the start: 2 copper layers, 34.3 x 39.4 mm, 39 parts, among them J1 USB2.0-C_SMT, J10 VBAT TH-2P, J2 VUSB PH-2P, J3 VUSB TH-2P, J4 3V3 PH-2P, J5 3V3 TH-2P, J6 VDD PH-2P, J7 VDD TH-2P, J8 VBAT PH-2P, J9 VBAT PH-2P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

Commit message: fix
Changed lines of the file:
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@@
 		(tags "resistor handsolder")
 		(property "Reference" "R8"
-			(at 1.778 1.651 0)
+			(at -2.794 0.127 0)
 			(layer "F.SilkS")
 			(effects
