File: test-lipo_battery/test-lipo_battery.kicad_sch (KiCad schematic)
At the start: 37 parts, among them J1 USB2.0-C_SMT, J10 VBAT TH-2P, J2 VUSB PH-2P, J3 VUSB TH-2P, J4 3V3 PH-2P, J5 3V3 TH-2P, J6 VDD PH-2P, J7 VDD TH-2P, J8 VBAT PH-2P, J9 VBAT PH-2P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

Commit message: fix
Other:
- note added: "MOSFETをDiodeの代わりとして使う場合の 接続が誤っていてたので MOSFETに意味はなし"
Changed lines of the file:
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@@
+		)
+	)
+	(text "MOSFETをDiodeの代わりとして使う場合の\n接続が誤っていてたので\nMOSFETに意味はなし"
+		(exclude_from_sim no)
+		(at 76.454 51.816 0)
+		(effects
+			(font
+				(size 1.27 1.27)
+			)
+			(justify left)
+		)
+	)
+	(text "MOSFETをDiodeの代わりとして使う場合の\n接続が誤っていてたので\nMOSFETに意味はなし"
+		(exclude_from_sim no)
+		(at 47.498 182.626 0)
+		(effects
+			(font
+				(size 1.27 1.27)
+			)
+			(justify left)
 		)
 	)
