File: grove_universal_board/grove_universal_board.kicad_sch (KiCad schematic)
At the start: 7 parts

Commit message: grove_universal_board/v1.1.0
Parts:
- added C1, C2: 10u, 74th:Capacitor_0603_1608, symbol Device:C
- added CH1, CH13, CH14, CH15, CH16, CH2, CH3, CH4, CH5, CH6, CH7, CH8, CH9: Pin_1, 74th:PinOut_Pin_3, symbol 74th_Interface:Pin_3
- added CH17: Pin_1, 74th:PinOut_Pin_3_Square, symbol 74th_Interface:Pin_3
- added JP1: Jumper_2_Open, 74th:SolderJumper-2, symbol 74th_Interface:Jumper_2
- added R1, R2: 1k, 74th:Register_0603_1608, symbol Device:R
- added U1: AMS1117, Package_TO_SOT_SMD:SOT-89-3, symbol 74th_Passive:AMS1117-3.3_Regulator_SOT89
- CH10: renamed from CH2; footprint 74th:PinOut_Universal-Board_bridge3 -> 74th:PinOut_Pin_2; symbol 74th_Interface:Pin_1 -> 74th_Interface:Pin_2
- CH11: renamed from CH3; footprint 74th:PinOut_Universal-Board_bridge3 -> 74th:PinOut_Pin_2; symbol 74th_Interface:Pin_1 -> 74th_Interface:Pin_2
- CH12: renamed from CH1; footprint 74th:PinOut_Universal-Board_bridge3 -> 74th:PinOut_Pin_4_GND; symbol 74th_Interface:Pin_1 -> 74th_Interface:Pin_4
- CH19: renamed from CH4; footprint 74th:PinOut_Universal-Board_bridge3 -> 74th:PinOut_Pin_3_Square; symbol 74th_Interface:Pin_1 -> 74th_Interface:Pin_3
- CH20: renamed from CH6; footprint 74th:PinOut_Universal-Board_bridge3 -> 74th:PinOut_Universal-Board_bridge6_with-Jumper; symbol 74th_Interface:Pin_1 -> 74th_Interface:Pin_6
- CH21: renamed from CH7; footprint 74th:PinOut_Universal-Board_bridge3 -> 74th:PinOut_Universal-Board_bridge6_with-Jumper_Square; symbol 74th_Interface:Pin_1 -> 74th_Interface:Pin_6
- renumbered CH5 to CH18
Connections:
- net D1/SDA: now reaches CH11.1, CH18.2 (SDA)
- net D1/SDA: now also CH11.2, CH12.2, R1.2
- net D0/SCL: now reaches CH10.1, CH18.1 (SCL)
- net D0/SCL: now also CH10.2, CH12.1, R2.2
- net GND: now reaches CH18.4 (GND), CH19.1, CH21.1
- net GND: now also CH12.4, CH19.2, CH19.3, CH21.2, CH21.3, CH21.4, CH21.5, CH21.6, C1.2, C2.2, CH17.1, CH17.2, CH17.3, U1.1 (GND)
- new net: CH8.1, CH8.2, CH8.3
- new net: CH7.1, CH7.2, CH7.3
- new net: CH6.1, CH6.2, CH6.3
- new net: CH16.1, CH16.2, CH16.3
- new net: CH2.1, CH2.2, CH2.3
- new net: CH4.1, CH4.2, CH4.3
- new net: CH5.1, CH5.2, CH5.3
- new net: CH13.1, CH13.2, CH13.3
- new net: CH14.1, CH14.2, CH14.3
- new net: CH3.1, CH3.2, CH3.3
- new net: CH1.1, CH1.2, CH1.3
- new net: CH9.1, CH9.2, CH9.3
- new net: CH15.1, CH15.2, CH15.3
- new net +5V: C2.1, CH12.3, CH18.3 (VCC), JP1.1 (A), U1.3 (VI)
- new net VCC: C1.1, CH20.1, CH20.2, CH20.3, CH20.4, CH20.5, CH20.6, JP1.2 (B), R1.1, R2.1, U1.2 (VO)
- no-connect marks 0 -> 2
Other:
- moved on the sheet: CH18
