File: usb_adapter_a-male_to_c-female/usb_adapter_a-male_to_c-female.kicad_pcb (KiCad board)
At the start: 2 copper layers, 16.5 x 14.5 mm, 5 parts, among them J1 USB_TypeA-2.0_Plug, J2 USB2.0-C_SMT, M2 Hole_M1.6_1.6

Commit message: usb-adapter-amcf/1.0.0
Parts:
- moved J2 1.36 mm to (76.9, 41.8)
- moved M2 1.30 mm to (78.0, 47.8)
- moved R1 0.91 mm to (70.7, 35.8)
- moved R2 0.57 mm to (70.9, 48.2)
Routing:
- net GND: track 6.16 -> 12.4 mm
- net Net-(J2-CC2): track 9.11 -> 6.69 mm
- net Net-(J1-VBUS): track 27.1 -> 25.5 mm, vias 1 -> 0
- net Net-(J1-D+): track 6.16 -> 4.70 mm
- net Net-(J1-D-): track 6.90 -> 5.46 mm
- net Net-(J2-CC1): track 9.52 -> 8.48 mm
Other:
- board size 16.5 x 14.5 mm -> 15.2 x 14.5 mm
- board text added: "AMCF"
- board text added: "USB"
- board text removed: "USB AMCF"
