File: usb_adapter_a-male_to_c-female/usb_adapter_a-male_to_c-female.kicad_sch (KiCad schematic)
At the start: 4 parts, among them J1 USB_TypeA-2.0_Plug, J2 USB2.0-C_SMT

Commit message: usb-adapter-amcf/1.0.0
Other:
- company: (none) -> Atsushi Morimoto (@74th)
- title: (none) -> USB AM-CF Adapter
Changed lines of the file:
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@@
 	(generator_version "8.0")
 	(paper "A4")
+	(title_block
+		(title "USB AM-CF Adapter")
+		(rev "v1.0.0")
+		(company "Atsushi Morimoto (@74th)")
+	)
 	(junction
 		(at 111.76 43.18)
