File: usb_adapter_micro-male_to_c-female/usb_adapter_micro-male_to_c-female.kicad_pcb (KiCad board)
At the start: 2 copper layers, 14 x 11.5 mm, 6 parts, among them J2 USB2.0-C_SMT, J3 USB_B_Micro

Commit message: usb-adapter-mmcf/1.0.1
Parts:
- turned R1 to 0 degrees
- turned R2 to 0 degrees
Connections:
- R1 pad 1: Net-(J2-VBUS) -> Net-(J2-CC2)
- R1 pad 2: Net-(J2-CC2) -> GND
- R2 pad 1: Net-(J2-VBUS) -> Net-(J2-CC1)
- R2 pad 2: Net-(J2-CC1) -> GND
Routing:
- net Net-(J2-VBUS): track 17.5 -> 13.1 mm, vias 2 -> 1
- net GND: track 0.00 -> 3.34 mm
Other:
- board text added: "v${REVISION}"
- board text removed: "v1.0.0"
