File: usb_adapter_micro-male_to_c-female/usb_adapter_micro-male_to_c-female.kicad_sch (KiCad schematic)
At the start: 6 parts, among them J2 USB2.0-C_SMT, J3 USB_B_Micro

Commit message: usb-adapter-mmcf/1.0.1
Connections:
- net GND: now also R1.2, R2.2
- net at J2.1 (VBUS), J3.1 (VBUS), R4.1: no longer R1.1, R2.1
- net at J2.5 (CC1): now also R2.1; no longer R2.2
- net at J2.6 (CC2): now also R1.1; no longer R1.2
Other:
- moved on the sheet: R1, R2
Changed lines of the file:
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@@
 	(title_block
 		(title "USB MM-CF Adapter")
-		(rev "v1.0.0")
+		(rev "v1.0.1")
 		(company "Atsushi Morimoto (@74th)")
-	)
-	(junction
-		(at 111.76 43.18)
-		(diameter 0)
-		(color 0 0 0 0)
-	)
-	(junction
-		(at 102.87 43.18)
-		(diameter 0)
-		(color 0 0 0 0)
 	)
 	(junction
@@
 	(wire
 		(pts
+			(xy 100.33 59.69) (xy 100.33 64.77)
+		)
+		(stroke
+			(width 0)
+			(type default)
+		)
+	)
+	(wire
+		(pts
 			(xy 50.8 50.8) (xy 129.54 50.8)
 		)
@@
 	(wire
 		(pts
-			(xy 111.76 64.77) (xy 124.46 64.77)
-		)
-		(stroke
-			(width 0)
-			(type default)
-		)
-	)
-	(wire
-		(pts
-			(xy 111.76 43.18) (xy 111.76 53.34)
+			(xy 100.33 59.69) (xy 129.54 59.69)
 		)
 		(stroke
@@
 	(wire
 		(pts
-			(xy 125.73 66.04) (xy 125.73 62.23)
-		)
-		(stroke
-			(width 0)
-			(type default)
-		)
-	)
-	(wire
-		(pts
-			(xy 125.73 62.23) (xy 129.54 62.23)
+			(xy 109.22 62.23) (xy 109.22 64.77)
 		)
 		(stroke
@@
 	(wire
 		(pts
-			(xy 124.46 59.69) (xy 129.54 59.69)
-		)
-		(stroke
-			(width 0)
-			(type default)
-		)
-	)
-	(wire
-		(pts
-			(xy 102.87 66.04) (xy 102.87 60.96)
-		)
-		(stroke
-			(width 0)
-			(type default)
-		)
-	)
-	(wire
-		(pts
-			(xy 111.76 43.18) (xy 129.54 43.18)
-		)
-		(stroke
-			(width 0)
-			(type default)
-		)
-	)
-	(wire
-		(pts
-			(xy 111.76 64.77) (xy 111.76 60.96)
+			(xy 63.5 43.18) (xy 129.54 43.18)
 		)
 		(stroke
@@
 	(wire
 		(pts
-			(xy 120.65 71.12) (xy 120.65 55.88)
+			(xy 120.65 72.39) (xy 120.65 55.88)
 		)
 		(stroke
@@
 	(wire
 		(pts
-			(xy 102.87 43.18) (xy 102.87 53.34)
-		)
-		(stroke
-			(width 0)
-			(type default)
-		)
-	)
-	(wire
-		(pts
-			(xy 63.5 43.18) (xy 102.87 43.18)
+			(xy 109.22 62.23) (xy 129.54 62.23)
 		)
 		(stroke
@@
 	(wire
 		(pts
-			(xy 102.87 66.04) (xy 125.73 66.04)
-		)
-		(stroke
-			(width 0)
-			(type default)
-		)
-	)
-	(wire
-		(pts
 			(xy 50.8 43.18) (xy 63.5 43.18)
 		)
@@
 	(wire
 		(pts
-			(xy 102.87 43.18) (xy 111.76 43.18)
-		)
-		(stroke
-			(width 0)
-			(type default)
-		)
-	)
-	(wire
-		(pts
 			(xy 63.5 64.77) (xy 63.5 63.5)
-		)
-		(stroke
-			(width 0)
-			(type default)
-		)
-	)
-	(wire
-		(pts
-			(xy 124.46 64.77) (xy 124.46 59.69)
 		)
 		(stroke
@@
 	)
 	(symbol
+		(lib_id "power:GND")
+		(at 100.33 72.39 0)
+		(unit 1)
+		(exclude_from_sim no)
+		(in_bom yes)
+		(on_board yes)
+		(dnp no)
+		(fields_autoplaced yes)
+		(property "Reference" "#PWR04"
+			(at 100.33 78.74 0)
+			(effects
+				(font
+					(size 1.27 1.27)
+				)
+				(hide yes)
+			)
+		)
+		(property "Value" "GND"
+			(at 100.33 77.47 0)
+			(effects
+				(font
+					(size 1.27 1.27)
+				)
+			)
+		)
+		(property "Footprint" ""
+			(at 100.33 72.39 0)
+			(effects
+				(font
+					(size 1.27 1.27)
+				)
+				(hide yes)
+			)
+		)
+		(property "Datasheet" ""
+			(at 100.33 72.39 0)
+			(effects
+				(font
+					(size 1.27 1.27)
+				)
+				(hide yes)
+			)
+		)
+		(property "Description" "Power symbol creates a global label with name \"GND\" , ground"
+			(at 100.33 72.39 0)
+			(effects
+				(font
+					(size 1.27 1.27)
+				)
+				(hide yes)
+			)
+		)
+		(pin "1"
+		)
+		(instances
+			(project "usb_adapter_micro-male_to_c-female"
+				(path "/9c4ea88e-8a29-402c-93bf-dd0d78f1062e"
+					(reference "#PWR04")
+					(unit 1)
+				)
+			)
+		)
+	)
+	(symbol
+		(lib_id "power:GND")
+		(at 109.22 72.39 0)
+		(unit 1)
+		(exclude_from_sim no)
+		(in_bom yes)
+		(on_board yes)
+		(dnp no)
+		(fields_autoplaced yes)
+		(property "Reference" "#PWR05"
+			(at 109.22 78.74 0)
+			(effects
+				(font
+					(size 1.27 1.27)
+				)
+				(hide yes)
+			)
+		)
+		(property "Value" "GND"
+			(at 109.22 77.47 0)
+			(effects
+				(font
+					(size 1.27 1.27)
+				)
+			)
+		)
+		(property "Footprint" ""
+			(at 109.22 72.39 0)
+			(effects
+				(font
+					(size 1.27 1.27)
+				)
+				(hide yes)
+			)
+		)
+		(property "Datasheet" ""
+			(at 109.22 72.39 0)
+			(effects
+				(font
+					(size 1.27 1.27)
+				)
+				(hide yes)
+			)
+		)
+		(property "Description" "Power symbol creates a global label with name \"GND\" , ground"
+			(at 109.22 72.39 0)
+			(effects
+				(font
+					(size 1.27 1.27)
+				)
+				(hide yes)
+			)
+		)
+		(pin "1"
+		)
+		(instances
+			(project "usb_adapter_micro-male_to_c-female"
+				(path "/9c4ea88e-8a29-402c-93bf-dd0d78f1062e"
+					(reference "#PWR05")
+					(unit 1)
+				)
+			)
+		)
+	)
+	(symbol
 		(lib_id "Connector:USB_B_Micro")
 		(at 43.18 48.26 0)
@@
 	(symbol
 		(lib_id "power:GND")
-		(at 120.65 71.12 0)
+		(at 120.65 72.39 0)
 		(unit 1)
 		(exclude_from_sim no)
@@
 		(fields_autoplaced yes)
 		(property "Reference" "#PWR02"
+			(at 120.65 78.74 0)
+			(effects
+				(font
+					(size 1.27 1.27)
+				)
+				(hide yes)
+			)
+		)
+		(property "Value" "GND"
 			(at 120.65 77.47 0)
 			(effects
@@
 					(size 1.27 1.27)
 				)
-				(hide yes)
-			)
-		)
-		(property "Value" "GND"
-			(at 120.65 76.2 0)
-			(effects
-				(font
-					(size 1.27 1.27)
-				)
 			)
 		)
 		(property "Footprint" ""
-			(at 120.65 71.12 0)
+			(at 120.65 72.39 0)
 			(effects
 				(font
@@
 		)
 		(property "Datasheet" ""
-			(at 120.65 71.12 0)
+			(at 120.65 72.39 0)
 			(effects
 				(font
@@
 		)
 		(property "Description" "Power symbol creates a global label with name \"GND\" , ground"
-			(at 120.65 71.12 0)
+			(at 120.65 72.39 0)
 			(effects
 				(font
@@
 	(symbol
 		(lib_id "Device:R")
-		(at 102.87 57.15 0)
+		(at 109.22 68.58 0)
 		(unit 1)
 		(exclude_from_sim no)
@@
 		(fields_autoplaced yes)
 		(property "Reference" "R1"
-			(at 105.41 55.8799 0)
+			(at 111.76 67.3099 0)
 			(effects
 				(font
@@
 		)
 		(property "Value" "56k"
-			(at 105.41 58.4199 0)
+			(at 111.76 69.8499 0)
 			(effects
 				(font
@@
 		)
 		(property "Footprint" "74th:Register_0603_1608"
-			(at 101.092 57.15 90)
+			(at 107.442 68.58 90)
 			(effects
 				(font
@@
 		)
 		(property "Datasheet" "~"
-			(at 102.87 57.15 0)
+			(at 109.22 68.58 0)
 			(effects
 				(font
@@
 		)
 		(property "Description" "Resistor"
-			(at 102.87 57.15 0)
+			(at 109.22 68.58 0)
 			(effects
 				(font
@@
 	(symbol
 		(lib_id "Device:R")
-		(at 111.76 57.15 0)
+		(at 100.33 68.58 0)
 		(unit 1)
 		(exclude_from_sim no)
@@
 		(fields_autoplaced yes)
 		(property "Reference" "R2"
-			(at 114.3 55.8799 0)
+			(at 102.87 67.3099 0)
 			(effects
 				(font
@@
 		)
 		(property "Value" "56k"
-			(at 114.3 58.4199 0)
+			(at 102.87 69.8499 0)
 			(effects
 				(font
@@
 		)
 		(property "Footprint" "74th:Register_0603_1608"
-			(at 109.982 57.15 90)
+			(at 98.552 68.58 90)
 			(effects
 				(font
@@
 		)
 		(property "Datasheet" "~"
-			(at 111.76 57.15 0)
+			(at 100.33 68.58 0)
 			(effects
 				(font
@@
 		)
 		(property "Description" "Resistor"
-			(at 111.76 57.15 0)
-			(effects
-				(font
+			(at 100.33 68.58 0)
+			(effects
+				(font
