File: usb_switch_adapter/usb_switch_adapter.kicad_sch (KiCad schematic)
At the start: 10 parts, among them J1 USB-C Plug, J2 USB2.0-C_SMT, SW1 SW_Push, U1 CH217K, U2 CH32V003J4M6

Commit message: usb-switch-adapter/1.0.0
Parts:
- U1: footprint Package_TO_SOT_SMD:SOT-23-6 -> 74th:Package_SOT-23-6
- U2: footprint Package_SO:SOIC-8_3.9x4.9mm_P1.27mm -> 74th:Package_SOIC-8_3.9x4.9mm_P1.27mm
Connections:
- net VBUS: now also J2.A4/B9 (VBUS), J2.A9/B4 (VBUS); no longer J1.A4 (VBUS), J1.A9 (VBUS), J1.B4 (VBUS), J1.B9 (VBUS)
- net VCC: now also J1.A4 (VBUS), J1.A9 (VBUS), J1.B4 (VBUS), J1.B9 (VBUS); no longer J2.A4/B9 (VBUS), J2.A9/B4 (VBUS)
Other:
- note added: "Downstream"
- note added: "Power Switch"
- note added: "Upstream"
- company: (none) -> Atsushi Morimoto (@74th)
- title: (none) -> USB Switch Adapter
- moved on the sheet: C1, CH1, D1, J1, J2, R1, R2, SW1, U1, U2

Commit message: usb-switch-adapter/1.1.0
Parts:
- CH1: value SWD 1Wire & UART TXD -> SWD 1Wire; footprint 74th:PinOut_Pin_4 -> 74th:PinOut_Pin_3_3GND; symbol 74th_Interface:SWD_WCH-1Wire_WITH-TXD-VCC -> 74th_Interface:SWD_WCH-1Wire_WITH-VCC
Connections:
- net GND: no longer D1.1 (K)
- net SWDIO: now also U2.8 (PD4/PD5/PD1/SWIO); no longer U2.7 (PC4)
- net SWITCH: now also U2.7 (PC4); no longer U2.8 (PD4/PD5/PD1/SWIO)
- net VBUS: now also R2.1
- net VCC: no longer R2.1
- net LED: now reaches U2.5 (PC1)
- net LED: now also D1.1 (K)
- net TXD: no longer names the net of U2.1 (PD6/PA1)
- net TXD: no longer CH1.4 (TXD)
Other:
- moved on the sheet: D1, R2, SW1
