File: 74TH-G054-grove_keymouse/grove_keymouse.kicad_sch (KiCad schematic)
At the start: 11 parts, among them J1 USB_TypeA-2.0_Plug, U1 CH9329, U2 CH213K

Commit message: Grove KeyMouse
Parts:
- D2: value LED -> Blue
Changed lines of the file:
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@@
 			)
 		)
-		(property "Value" "LED"
+		(property "Value" "Blue"
 			(at 262.89 57.4674 90)
 			(effects
