File: MISC-usb_adapter_micro-male_to_c-female/usb_adapter_micro-male_to_c-female.kicad_sch (KiCad schematic)
At the start: 6 parts, among them J2 USB2.0-C_SMT, J3 USB_B_Micro

Commit message: usb_adapter_micro-male_to_c-female/1.0.0
Connections:
- net at J2.2 (D-): now also J3.2 (D-); no longer J3.3 (D+)
- net at J2.3 (D+): now also J3.3 (D+); no longer J3.2 (D-)
Changed lines of the file:
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@@
 	(title_block
 		(title "USB MM-CF Adapter")
-		(rev "v1.0.1")
+		(rev "v1.0.2")
 		(company "Atsushi Morimoto (@74th)")
 	)
@@
 	(wire
 		(pts
-			(xy 50.8 50.8) (xy 129.54 50.8)
-		)
-		(stroke
-			(width 0)
-			(type default)
-		)
-	)
-	(wire
-		(pts
 			(xy 100.33 59.69) (xy 129.54 59.69)
 		)
@@
 	(wire
 		(pts
+			(xy 91.44 50.8) (xy 50.8 50.8)
+		)
+		(stroke
+			(width 0)
+			(type default)
+		)
+	)
+	(wire
+		(pts
 			(xy 54.61 53.34) (xy 54.61 64.77)
 		)
@@
 	(wire
 		(pts
+			(xy 50.8 48.26) (xy 93.98 48.26)
+		)
+		(stroke
+			(width 0)
+			(type default)
+		)
+	)
+	(wire
+		(pts
 			(xy 63.5 43.18) (xy 129.54 43.18)
 		)
@@
 	(wire
 		(pts
-			(xy 50.8 48.26) (xy 129.54 48.26)
+			(xy 96.52 53.34) (xy 91.44 53.34)
 		)
 		(stroke
@@
 	(wire
 		(pts
+			(xy 129.54 48.26) (xy 96.52 48.26)
+		)
+		(stroke
+			(width 0)
+			(type default)
+		)
+	)
+	(wire
+		(pts
+			(xy 93.98 48.26) (xy 93.98 50.8)
+		)
+		(stroke
+			(width 0)
+			(type default)
+		)
+	)
+	(wire
+		(pts
+			(xy 93.98 50.8) (xy 129.54 50.8)
+		)
+		(stroke
+			(width 0)
+			(type default)
+		)
+	)
+	(wire
+		(pts
+			(xy 96.52 48.26) (xy 96.52 53.34)
+		)
+		(stroke
+			(width 0)
+			(type default)
+		)
+	)
+	(wire
+		(pts
 			(xy 63.5 64.77) (xy 63.5 63.5)
 		)
 		(stroke
+			(width 0)
+			(type default)
+		)
+	)
+	(wire
+		(pts
+			(xy 91.44 53.34) (xy 91.44 50.8)
+		)
+		(stroke
