File: 74TH-G060-7seg-grove/74TH-G060-7seg-grove.kicad_sch (KiCad schematic)
At the start: 26 parts, among them U1 CH32V003F4P6, U2 OSL10561-LW, U3 OSL10561-LW, U4 OSL10561-LW, U5 OSL10561-LW, U6 AMS1117, U7 CH213K

Commit message: 7seg-grove/1.0.0
Parts:
- renumbered C3 to C2, C2 to C3, CH2 to CH1, CH1 to CH2, R9 to R1, R7 to R2, R5 to R3, R1 to R5, R8 to R6, R6 to R7, R2 to R8, R3 to R9, U2 to U1, U3 to U2, U4 to U3, U5 to U4, U1 to U5, U7 to U6, U6 to U7
Changed lines of the file:
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@@
 		(dnp no)
 		(fields_autoplaced yes)
-		(property "Reference" "R9"
+		(property "Reference" "R1"
 			(at 115.57 144.78 90)
 			(effects
@@
 			(project "74TH-G060-7seg-grove"
 				(path "/e0a12cc3-fc1c-4902-9f3a-6460933c3c18"
-					(reference "R9")
+					(reference "R1")
 					(unit 1)
 				)
@@
 		(dnp no)
 		(fields_autoplaced yes)
-		(property "Reference" "R3"
+		(property "Reference" "R9"
 			(at 123.19 123.19 90)
 			(effects
@@
 			(project "74TH-G060-7seg-grove"
 				(path "/e0a12cc3-fc1c-4902-9f3a-6460933c3c18"
-					(reference "R3")
+					(reference "R9")
 					(unit 1)
 				)
@@
 		(dnp no)
 		(fields_autoplaced yes)
-		(property "Reference" "C2"
+		(property "Reference" "C3"
 			(at 58.42 97.7899 0)
 			(effects
@@
 			(project "74TH-G060-7seg-grove"
 				(path "/e0a12cc3-fc1c-4902-9f3a-6460933c3c18"
-					(reference "C2")
+					(reference "C3")
 					(unit 1)
 				)
@@
 		(dnp no)
 		(fields_autoplaced yes)
-		(property "Reference" "R5"
+		(property "Reference" "R3"
 			(at 116.84 154.94 90)
 			(effects
@@
 			(project "74TH-G060-7seg-grove"
 				(path "/e0a12cc3-fc1c-4902-9f3a-6460933c3c18"
-					(reference "R5")
+					(reference "R3")
 					(unit 1)
 				)
@@
 		(dnp no)
 		(fields_autoplaced yes)
-		(property "Reference" "R1"
+		(property "Reference" "R5"
 			(at 116.84 163.83 90)
 			(effects
@@
 			(project "74TH-G060-7seg-grove"
 				(path "/e0a12cc3-fc1c-4902-9f3a-6460933c3c18"
-					(reference "R1")
+					(reference "R5")
 					(unit 1)
 				)
@@
 		(dnp no)
 		(fields_autoplaced yes)
-		(property "Reference" "CH1"
+		(property "Reference" "CH2"
 			(at 30.48 37.4649 0)
 			(effects
@@
 			(project ""
 				(path "/e0a12cc3-fc1c-4902-9f3a-6460933c3c18"
-					(reference "CH1")
+					(reference "CH2")
 					(unit 1)
 				)
@@
 		(dnp no)
 		(fields_autoplaced yes)
-		(property "Reference" "U5"
+		(property "Reference" "U4"
 			(at 242.57 82.55 0)
 			(effects
@@
 			(project "74TH-G060-7seg-grove"
 				(path "/e0a12cc3-fc1c-4902-9f3a-6460933c3c18"
-					(reference "U5")
+					(reference "U4")
 					(unit 1)
 				)
@@
 		(dnp no)
 		(fields_autoplaced yes)
-		(property "Reference" "U3"
+		(property "Reference" "U2"
 			(at 242.57 31.75 0)
 			(effects
@@
 			(project "74TH-G060-7seg-grove"
 				(path "/e0a12cc3-fc1c-4902-9f3a-6460933c3c18"
-					(reference "U3")
+					(reference "U2")
 					(unit 1)
 				)
@@
 		(dnp no)
 		(fields_autoplaced yes)
-		(property "Reference" "U2"
+		(property "Reference" "U1"
 			(at 187.96 31.75 0)
 			(effects
@@
 			(project ""
 				(path "/e0a12cc3-fc1c-4902-9f3a-6460933c3c18"
-					(reference "U2")
+					(reference "U1")
 					(unit 1)
 				)
@@
 		(dnp no)
 		(fields_autoplaced yes)
-		(property "Reference" "R7"
+		(property "Reference" "R2"
 			(at 34.29 176.53 90)
 			(effects
@@
 			(project "74TH-G060-7seg-grove"
 				(path "/e0a12cc3-fc1c-4902-9f3a-6460933c3c18"
-					(reference "R7")
+					(reference "R2")
 					(unit 1)
 				)
@@
 		(dnp no)
 		(fields_autoplaced yes)
-		(property "Reference" "U1"
+		(property "Reference" "U5"
 			(at 75.8541 142.24 0)
 			(effects
@@
 			(project ""
 				(path "/e0a12cc3-fc1c-4902-9f3a-6460933c3c18"
-					(reference "U1")
+					(reference "U5")
 					(unit 1)
 				)
@@
 		(dnp no)
 		(fields_autoplaced yes)
-		(property "Reference" "R2"
+		(property "Reference" "R8"
 			(at 34.29 125.73 90)
 			(effects
@@
 			(project "74TH-G060-7seg-grove"
 				(path "/e0a12cc3-fc1c-4902-9f3a-6460933c3c18"
-					(reference "R2")
+					(reference "R8")
 					(unit 1)
 				)
@@
 		(dnp no)
 		(fields_autoplaced yes)
-		(property "Reference" "R6"
+		(property "Reference" "R7"
 			(at 34.29 186.69 90)
 			(effects
@@
 			(project "74TH-G060-7seg-grove"
 				(path "/e0a12cc3-fc1c-4902-9f3a-6460933c3c18"
-					(reference "R6")
+					(reference "R7")
 					(unit 1)
 				)
@@
 		(dnp no)
 		(fields_autoplaced yes)
-		(property "Reference" "R8"
+		(property "Reference" "R6"
 			(at 34.29 166.37 90)
 			(effects
@@
 			(project "74TH-G060-7seg-grove"
 				(path "/e0a12cc3-fc1c-4902-9f3a-6460933c3c18"
-					(reference "R8")
+					(reference "R6")
 					(unit 1)
 				)
@@
 		(dnp no)
 		(fields_autoplaced yes)
-		(property "Reference" "U6"
+		(property "Reference" "U7"
 			(at 69.85 88.9 0)
 			(effects
@@
 			(project ""
 				(path "/e0a12cc3-fc1c-4902-9f3a-6460933c3c18"
-					(reference "U6")
+					(reference "U7")
 					(unit 1)
 				)
@@
 		(dnp no)
 		(fields_autoplaced yes)
-		(property "Reference" "U4"
+		(property "Reference" "U3"
 			(at 187.96 78.74 0)
 			(effects
@@
 			(project "74TH-G060-7seg-grove"
 				(path "/e0a12cc3-fc1c-4902-9f3a-6460933c3c18"
-					(reference "U4")
+					(reference "U3")
 					(unit 1)
 				)
@@
 		(dnp no)
 		(fields_autoplaced yes)
-		(property "Reference" "U7"
+		(property "Reference" "U6"
 			(at 102.235 76.2 0)
 			(effects
@@
 			(project ""
 				(path "/e0a12cc3-fc1c-4902-9f3a-6460933c3c18"
-					(reference "U7")
+					(reference "U6")
 					(unit 1)
 				)
@@
 		(dnp no)
 		(fields_autoplaced yes)
-		(property "Reference" "C3"
+		(property "Reference" "C2"
 			(at 87.63 97.7899 0)
 			(effects
@@
 			(project "74TH-G060-7seg-grove"
 				(path "/e0a12cc3-fc1c-4902-9f3a-6460933c3c18"
-					(reference "C3")
+					(reference "C2")
 					(unit 1)
 				)
@@
 		(dnp no)
 		(fields_autoplaced yes)
-		(property "Reference" "CH2"
+		(property "Reference" "CH1"
 			(at 168.91 140.97 0)
 			(effects
@@
 			(project ""
 				(path "/e0a12cc3-fc1c-4902-9f3a-6460933c3c18"
-					(reference "CH2")
-					(unit 1)
-				)
+					(reference "CH1")
+					(unit 1)
+				)

Commit message: 7seg-grove/1.0.0
Parts:
- CH2: footprint 74th:Connector_HY-2.0_SMD_4Pin -> 74th:Connector_Grove_or_Qwiic
Changed lines of the file:
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@@
 			)
 		)
-		(property "Footprint" "74th:Connector_HY-2.0_SMD_4Pin"
+		(property "Footprint" "74th:Connector_Grove_or_Qwiic"
 			(at 53.34 46.99 0)
 			(effects

Commit message: fix
Connections:
- net SA: now also R1.2, U1.7 (A), U2.7 (A), U3.7 (A), U4.7 (A); no longer R2.1, U1.10 (A), U2.10 (A), U3.10 (A), U4.10 (A)
- net SB: now also R5.2, U1.6 (B), U2.6 (B), U3.6 (B), U4.6 (B); no longer R6.1, U1.9 (B), U2.9 (B), U3.9 (B), U4.9 (B)
- net SC: now also R8.1, U1.4 (C), U2.4 (C), U3.4 (C), U4.4 (C); no longer R1.2, U1.7 (C), U2.7 (C), U3.7 (C), U4.7 (C)
- net SD: now also R3.2, U1.2 (D), U2.2 (D), U3.2 (D), U4.2 (D); no longer R4.2, U1.5 (D), U2.5 (D), U3.5 (D), U4.5 (D)
- net SDP: now also R4.2, U1.5 (DP), U2.5 (DP), U3.5 (DP), U4.5 (DP); no longer R5.2, U1.6 (DP), U2.6 (DP), U3.6 (DP), U4.6 (DP)
- net SE: now also R7.1, U1.1 (E), U2.1 (E), U3.1 (E), U4.1 (E); no longer R8.1, U1.4 (E), U2.4 (E), U3.4 (E), U4.4 (E)
- net SF: now also R6.1, U1.9 (F), U2.9 (F), U3.9 (F), U4.9 (F); no longer R3.2, U1.2 (F), U2.2 (F), U3.2 (F), U4.2 (F)
- net SG: now also R2.1, U1.10 (G), U2.10 (G), U3.10 (G), U4.10 (G); no longer R7.1, U1.1 (G), U2.1 (G), U3.1 (G), U4.1 (G)
- net SW1 renamed SEL4
- net SW2 renamed SEL3
- net SW3 renamed SEL2
- net SW4 renamed SEL1
Changed lines of the file:
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@@
+	(wire
+		(pts
+			(xy 21.59 182.88) (xy 30.48 182.88)
+		)
+		(stroke
+			(width 0)
+			(type default)
+		)
+	)
 	(wire
 		(pts
@@
 		(pts
 			(xy 39.37 157.48) (xy 50.8 157.48)
-		)
-		(stroke
-			(width 0)
-			(type default)
-		)
-	)
-	(wire
-		(pts
-			(xy 21.59 182.88) (xy 30.48 182.88)
 		)
 		(stroke
@@
 		)
 	)
-	(label "SW4"
+	(label "SEL1"
 		(at 265.43 110.49 180)
 		(fields_autoplaced yes)
@@
 	)
 	(label "SA"
-		(at 21.59 182.88 0)
-		(fields_autoplaced yes)
-		(effects
-			(font
-				(size 1.27 1.27)
-			)
-			(justify left bottom)
+		(at 128.27 151.13 180)
+		(fields_autoplaced yes)
+		(effects
+			(font
+				(size 1.27 1.27)
+			)
+			(justify right bottom)
 		)
 	)
@@
 		)
 	)
-	(label "SW1"
+	(label "SEL4"
 		(at 106.68 167.64 180)
 		(fields_autoplaced yes)
@@
 		)
 	)
-	(label "SW1"
+	(label "SEL4"
 		(at 209.55 59.69 180)
 		(fields_autoplaced yes)
@@
 	)
 	(label "SB"
-		(at 21.59 172.72 0)
-		(fields_autoplaced yes)
-		(effects
-			(font
-				(size 1.27 1.27)
-			)
-			(justify left bottom)
+		(at 130.81 170.18 180)
+		(fields_autoplaced yes)
+		(effects
+			(font
+				(size 1.27 1.27)
+			)
+			(justify right bottom)
 		)
 	)
@@
 	)
 	(label "SC"
-		(at 128.27 151.13 180)
-		(fields_autoplaced yes)
-		(effects
-			(font
-				(size 1.27 1.27)
-			)
-			(justify right bottom)
+		(at 22.86 132.08 0)
+		(fields_autoplaced yes)
+		(effects
+			(font
+				(size 1.27 1.27)
+			)
+			(justify left bottom)
 		)
 	)
@@
 		)
 	)
-	(label "SW3"
+	(label "SEL2"
 		(at 209.55 106.68 180)
 		(fields_autoplaced yes)
@@
 		)
 	)
-	(label "SW4"
+	(label "SEL1"
 		(at 43.18 162.56 0)
 		(fields_autoplaced yes)
@@
 		)
 	)
-	(label "SW2"
+	(label "SEL3"
 		(at 43.18 165.1 0)
 		(fields_autoplaced yes)
@@
 	)
 	(label "SE"
-		(at 22.86 132.08 0)
+		(at 21.59 193.04 0)
 		(fields_autoplaced yes)
 		(effects
@@
 	)
 	(label "SG"
-		(at 21.59 193.04 0)
+		(at 21.59 182.88 0)
 		(fields_autoplaced yes)
 		(effects
@@
 	)
 	(label "SD"
-		(at 128.27 139.7 180)
+		(at 129.54 161.29 180)
 		(fields_autoplaced yes)
 		(effects
@@
 	)
 	(label "SDP"
-		(at 130.81 170.18 180)
-		(fields_autoplaced yes)
-		(effects
-			(font
-				(size 1.27 1.27)
-			)
-			(justify right bottom)
-		)
-	)
-	(label "SW3"
+		(at 128.27 139.7 180)
+		(fields_autoplaced yes)
+		(effects
+			(font
+				(size 1.27 1.27)
+			)
+			(justify right bottom)
+		)
+	)
+	(label "SEL2"
 		(at 43.18 160.02 0)
 		(fields_autoplaced yes)
@@
 	)
 	(label "SF"
-		(at 129.54 161.29 180)
-		(fields_autoplaced yes)
-		(effects
-			(font
-				(size 1.27 1.27)
-			)
-			(justify right bottom)
+		(at 21.59 172.72 0)
+		(fields_autoplaced yes)
+		(effects
+			(font
+				(size 1.27 1.27)
+			)
+			(justify left bottom)
 		)
 	)
@@
 		)
 	)
-	(label "SW2"
+	(label "SEL3"
 		(at 264.16 59.69 180)
 		(fields_autoplaced yes)

Commit message: update README
Other:
- title: (none) -> 7Seg Grove
Changed lines of the file:
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@@
 	(generator_version "8.0")
 	(paper "A4")
+	(title_block
+		(title "7Seg Grove")
+		(rev "1.0.1")
+	)
 	(junction
 		(at 254 59.69)
