File: 74TH-G060-7seg-grove/74TH-G060-7seg-grove.kicad_sch (KiCad schematic)
At the start: 26 parts, among them U1 OSL10561-LW, U2 OSL10561-LW, U3 OSL10561-LW, U4 OSL10561-LW, U5 CH32V003F4P6, U6 CH213K, U7 AMS1117

Commit message: up
Connections:
- net SA: now also R1.1; no longer R1.2
- net SC: now also R8.2; no longer R8.1
- net SDP: now also R4.1; no longer R4.2
- net SEL1: now also U5.16 (PC6/SPI_MOSI); no longer U5.3 (PD6/UART_RX/ADC6)
- net SEL2: now also U5.15 (PC5/SPI_SCK); no longer U5.2 (PD5/UART_TX/ADC5)
- net SEL3: now also U5.17 (PC7/SPI_MISO); no longer U5.1 (PD4/UART_CK/ADC7)
- net SEL4: now also U5.5 (PA1/ADC1/OSC_IN); no longer U5.10 (PC0)
- net SWDIO: now also R3.1
- net at U5.14 (PC4/ADC2): no longer R1.1
- net at U5.19 (PD2/ADC3): now also R8.1; no longer R3.1
- net at R5.1: now also U5.8 (PD0); no longer U5.13 (PC3)
- net at R2.2: now also U5.2 (PD5/UART_TX/ADC5); no longer U5.16 (PC6/SPI_MOSI)
- net at R6.2: now also U5.3 (PD6/UART_RX/ADC6); no longer U5.15 (PC5/SPI_SCK)
- net at R7.2: now also U5.1 (PD4/UART_CK/ADC7); no longer U5.17 (PC7/SPI_MISO)
- net at U5.20 (PD3/UART_CTS/ADC4): now also R4.2; no longer R8.2
- net at U5.4 (PD7/NRST): now also R1.2
- no-connect marks 2 -> 3
Other:
- moved on the sheet: R1, R2, R3, R4, R5, R6, R7, R8
