File: 74TH-G060-7seg-grove/74TH-G060-7seg-grove.kicad_pcb (KiCad board)
At the start: 2 copper layers, 70 x 20.5 mm, 31 parts, among them M2 Hole_M2_2.2-TH, U1 CH32V003F4P6, U2 OSL10561-LW, U3 OSL10561-LW, U4 OSL10561-LW, U5 OSL10561-LW, U6 AMS1117, U7 CH213K

Commit message: 7seg-grove/1.0.0
Parts:
- CH2: renamed from CH1; footprint 74th:Connector_HY-2.0_SMD_4Pin -> 74th:Connector_Grove_or_Qwiic
- renumbered C3 to C2, C2 to C3, CH2 to CH1, M2 to M1, M2 to M3, M2 to M4, R9 to R1, R7 to R2, R5 to R3, R1 to R5, R8 to R6, R6 to R7, R2 to R8, R3 to R9, U2 to U1, U3 to U2, U4 to U3, U5 to U4, U1 to U5, U7 to U6, U6 to U7
Routing:
- net GND: track 15.8 -> 14.7 mm, vias 40 -> 36

Commit message: fix
Parts:
- moved CH2 1.00 mm to (45.0, 47.6)
- moved M1 1.00 mm to (37.8, 39.8)
- moved M2 1.00 mm to (37.8, 55.8)
- moved M3 1.00 mm to (105.2, 39.8)
- moved M4 1.00 mm to (105.2, 55.5)
Connections:
- net /SW1 renamed /SEL4
- net /SW2 renamed /SEL3
- net /SW3 renamed /SEL2
- net /SW4 renamed /SEL1
- R1 pad 2: /SC -> /SA
- R2 pad 1: /SA -> /SG
- R3 pad 2: /SF -> /SD
- R4 pad 2: /SD -> /SDP
- R5 pad 2: /SDP -> /SB
- R6 pad 1: /SB -> /SF
- R7 pad 1: /SG -> /SE
- R8 pad 1: /SE -> /SC
- U1 pad 1: /SG -> /SE
- U1 pad 10: /SA -> /SG
- U1 pad 2: /SF -> /SD
- U1 pad 4: /SE -> /SC
- U1 pad 5: /SD -> /SDP
- U1 pad 6: /SDP -> /SB
- U1 pad 7: /SC -> /SA
- U1 pad 9: /SB -> /SF
- U2 pad 1: /SG -> /SE
- U2 pad 10: /SA -> /SG
- U2 pad 2: /SF -> /SD
- U2 pad 4: /SE -> /SC
- U2 pad 5: /SD -> /SDP
- U2 pad 6: /SDP -> /SB
- U2 pad 7: /SC -> /SA
- U2 pad 9: /SB -> /SF
- U3 pad 1: /SG -> /SE
- U3 pad 10: /SA -> /SG
- U3 pad 2: /SF -> /SD
- U3 pad 4: /SE -> /SC
- U3 pad 5: /SD -> /SDP
- U3 pad 6: /SDP -> /SB
- U3 pad 7: /SC -> /SA
- U3 pad 9: /SB -> /SF
- U4 pad 1: /SG -> /SE
- U4 pad 10: /SA -> /SG
- U4 pad 2: /SF -> /SD
- U4 pad 4: /SE -> /SC
- U4 pad 5: /SD -> /SDP
- U4 pad 6: /SDP -> /SB
- U4 pad 7: /SC -> /SA
- U4 pad 9: /SB -> /SF
Routing:
- net /SD: track 48.9 -> 55.0 mm, vias 2 -> 4
- net /SA: track 55.4 -> 50.2 mm
- net /SB: track 54.6 -> 50.8 mm, vias 5 -> 1
- net /SE: track 51.5 -> 55.0 mm
- net /SCL: track 41.1 -> 44.2 mm
- net GND: track 14.7 -> 17.5 mm
- net /SDP: track 50.8 -> 48.9 mm, vias 1 -> 2
- net /SDA: track 43.0 -> 41.3 mm
- net /SC: track 50.3 -> 51.5 mm
- net /SF: track 55.0 -> 54.6 mm, vias 4 -> 5
Other:
- board size 70 x 20.5 mm -> 72 x 20.5 mm

Commit message: update README
Parts:
- moved CH2 0.52 mm to (45.5, 47.8)
- moved M1 0.50 mm to (38.2, 39.8)
- moved M2 0.50 mm to (38.2, 55.8)
Routing:
- net /SCL: track 44.2 -> 41.4 mm
- net GND: track 17.5 -> 19.0 mm
Other:
- board size 72 x 20.5 mm -> 71.5 x 20.5 mm

Commit message: update README
Parts:
- moved M3 1.00 mm to (104.2, 39.8)
- moved M4 1.00 mm to (104.2, 55.5)
- moved CH2 0.50 mm to (46.0, 47.8)
- moved M1 0.50 mm to (38.8, 39.8)
- moved M2 0.50 mm to (38.8, 55.8)
Routing:
- net GND: track 19.0 -> 21.3 mm
- net /SDA: track 41.6 -> 42.7 mm
Other:
- board size 71.5 x 20.5 mm -> 70 x 20.5 mm

Commit message: update
Other:
- board text added: "3V3"
- board text added: "GND"
- board text added: "SCL"
- board text added: "SDA"
- board text added: "SWDIO"
- board text added: "VCC"
Changed lines of the file:
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@@
 		(at 48.82 39.3 180)
 		(property "Reference" "CH3"
-			(at 0.22 -2.2 0)
+			(at -3.28 0.9 0)
 			(unlocked yes)
 			(layer "B.SilkS")
@@
 		)
 	)
+	(gr_line
+		(start 49.2 40.6)
+		(end 48.9 40.3)
+		(stroke
+			(width 0.15)
+			(type default)
+		)
+		(layer "B.SilkS")
+	)
+	(gr_line
+		(start 48.9 41.7)
+		(end 48.9 40.3)
+		(stroke
+			(width 0.15)
+			(type default)
+		)
+		(layer "B.SilkS")
+	)
+	(gr_line
+		(start 48.6 40.6)
+		(end 48.9 40.3)
+		(stroke
+			(width 0.15)
+			(type default)
+		)
+		(layer "B.SilkS")
+	)
+	(gr_line
+		(start 51.8 41.7)
+		(end 48.9 41.7)
+		(stroke
+			(width 0.15)
+			(type default)
+		)
+		(layer "B.SilkS")
+	)
 	(gr_arc
 		(start 106.5 56)
@@
 		(layer "Edge.Cuts")
 	)
+	(gr_text "SWDIO"
+		(at 45.4 55.4 45)
+		(layer "B.SilkS")
+		(effects
+			(font
+				(size 1 1)
+				(thickness 0.14)
+			)
+			(justify right mirror)
+		)
+	)
 	(gr_text "7Seg Grove"
 		(at 104.8 45.4 0)
@@
 		)
 	)
+	(gr_text "SDA"
+		(at 54.2 43.2 0)
+		(layer "B.SilkS")
+		(effects
+			(font
+				(size 1 1)
+				(thickness 0.14)
+			)
+			(justify left mirror)
+		)
+	)
+	(gr_text "3V3"
+		(at 43.2 55.6 45)
+		(layer "B.SilkS")
+		(effects
+			(font
+				(size 1 1)
+				(thickness 0.14)
+			)
+			(justify right mirror)
+		)
+	)
 	(gr_text "C"
 		(at 50 38.9 0)
@@
 		)
 	)
+	(gr_text "SCL"
+		(at 54.9 41.8 0)
+		(layer "B.SilkS")
+		(effects
+			(font
+				(size 1 1)
+				(thickness 0.14)
+			)
+			(justify left mirror)
+		)
+	)
+	(gr_text "GND"
+		(at 47.8 55.3 45)
+		(layer "B.SilkS")
+		(effects
+			(font
+				(size 1 1)
+				(thickness 0.14)
+			)
+			(justify right mirror)
+		)
+	)
 	(gr_text "G"
 		(at 42.5 38.9 0)
@@
 		)
 	)
+	(gr_text "GND"
+		(at 52.4 46 0)
+		(layer "B.SilkS")
+		(effects
+			(font
+				(size 1 1)
+				(thickness 0.14)
+			)
+			(justify left mirror)
+		)
+	)
 	(gr_text "74TH-G060-${REVISION}"
 		(at 89.3 53.6 0)
@@
 		)
 	)
+	(gr_text "VCC"
+		(at 53.3 44.6 0)
+		(layer "B.SilkS")
+		(effects
+			(font
+				(size 1 1)
+				(thickness 0.14)
+			)
+			(justify left mirror)
+		)
+	)

Commit message: up
Parts:
- turned R1 to 180 degrees
- turned R4 to 180 degrees
- turned R8 to 0 degrees
Connections:
- R1 pad 1: Net-(U5-PC4/ADC2) -> /SA
- R1 pad 2: /SA -> Net-(U5-PD7/NRST)
- R2 pad 2: Net-(U5-PC6/SPI_MOSI) -> Net-(U5-PD5/UART_TX/ADC5)
- R3 pad 1: Net-(U5-PD2/ADC3) -> /SWDIO
- R4 pad 1: Net-(U5-PA1/ADC1/OSC_IN) -> /SDP
- R4 pad 2: /SDP -> Net-(U5-PD3/UART_CTS/ADC4)
- R5 pad 1: Net-(U5-PC3) -> Net-(U5-PD0)
- R6 pad 2: Net-(U5-PC5/SPI_SCK) -> Net-(U5-PD6/UART_RX/ADC6)
- R7 pad 2: Net-(U5-PC7/SPI_MISO) -> Net-(U5-PD4/UART_CK/ADC7)
- R8 pad 1: /SC -> Net-(U5-PD2/ADC3)
- R8 pad 2: Net-(U5-PD3/UART_CTS/ADC4) -> /SC
- U5 pad 1: /SEL3 -> Net-(U5-PD4/UART_CK/ADC7)
- U5 pad 10: /SEL4 -> unconnected-(U5-PC0-Pad10)
- U5 pad 13: Net-(U5-PC3) -> unconnected-(U5-PC3-Pad13)
- U5 pad 14: Net-(U5-PC4/ADC2) -> unconnected-(U5-PC4/ADC2-Pad14)
- U5 pad 15: Net-(U5-PC5/SPI_SCK) -> /SEL2
- U5 pad 16: Net-(U5-PC6/SPI_MOSI) -> /SEL1
- U5 pad 17: Net-(U5-PC7/SPI_MISO) -> /SEL3
- U5 pad 2: /SEL2 -> Net-(U5-PD5/UART_TX/ADC5)
- U5 pad 3: /SEL1 -> Net-(U5-PD6/UART_RX/ADC6)
- U5 pad 4: unconnected-(U5-PD7/NRST-Pad4) -> Net-(U5-PD7/NRST)
- U5 pad 5: Net-(U5-PA1/ADC1/OSC_IN) -> /SEL4
- U5 pad 8: unconnected-(U5-PD0-Pad8) -> Net-(U5-PD0)
Routing:
- net Net-(U5-PA1/ADC1/OSC_IN): track 18.9 -> 0.00 mm
- net Net-(U5-PD5/UART_TX/ADC5): track 0.00 -> 18.2 mm, vias 0 -> 2
- net Net-(U5-PD7/NRST): track 0.00 -> 17.0 mm, vias 0 -> 2
- net Net-(U5-PD4/UART_CK/ADC7): track 0.00 -> 13.7 mm, vias 0 -> 2
- net Net-(U5-PD6/UART_RX/ADC6): track 0.00 -> 13.0 mm, vias 0 -> 2
- net /SEL3: track 29.4 -> 17.2 mm, vias 2 -> 1
- net Net-(U5-PD0): track 0.00 -> 11.3 mm, vias 0 -> 2
- net Net-(U5-PC4/ADC2): track 9.85 -> 0.00 mm
- net Net-(U5-PC6/SPI_MOSI): track 9.73 -> 0.00 mm
- net /SWDIO: track 26.4 -> 36.0 mm
- net Net-(U5-PC3): track 5.28 -> 0.00 mm
- net Net-(U5-PC5/SPI_SCK): track 5.16 -> 0.00 mm
- net Net-(U5-PC7/SPI_MISO): track 5.04 -> 0.00 mm
- net Net-(U5-PD2/ADC3): track 9.87 -> 4.91 mm
- net Net-(U5-PD3/UART_CTS/ADC4): track 5.18 -> 9.50 mm
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