File: 74TH-G065-wifi_keymouse/74TH-G065-wifi_keymouse.kicad_pcb (KiCad board)
At the start: 2 copper layers, 20 x 41.5 mm, 23 parts, among them J1 USB_TypeA-2.0_Plug, J2 ESP-Prog-ProgramCOM_RECV, J3 ESP-Prog-ProgramCOM_RECV_Stra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, M2 Hole_M2_2.0, SW1 SW_Push, U1 CH9329, U2 ESP32-C3-WROOM-02, U3 CH217K, U4 AMS1117

Commit message: wifi_keymouse/1.0.0
Parts:
- removed J2: ESP-Prog-ProgramCOM_RECV, 74th:Connector_BoxPinHeader_2x03_P1.27mm
- added CH1: Pin_5, 74th:PinOut_Pin_5_GND, F.Cu at (0.76, 0.76)
- added R10: 5.1k, 74th:Register_0603_1608, B.Cu at (64.4, 64.3)
- added R7: 10, 74th:Register_0603_1608, B.Cu at (65.6, 51.8)
- added R8: 10, 74th:Register_0603_1608, B.Cu at (65.6, 50.3)
- added R9: 5.1k, 74th:Register_0603_1608, B.Cu at (64.3, 66.2)
- J3: value ESP-Prog-ProgramCOM_RECV_Straight -> USB2.0-C_SMT; footprint 74th:PinOut_Pin_6_GND -> 74th:Connector_USB-C-Receptacle_SMT_12-Pin_Simple
- R6: moved to B.Cu
- moved J3 18.0 mm to (52.6, 64.1), turned to -90 degrees
- moved R6 14.4 mm to (67.9, 66.2), turned to 0 degrees
- moved D1 8.81 mm to (65.5, 61.2)
- moved SW1 8.78 mm to (65.9, 65.4), turned to 180 degrees
- moved R5 8.11 mm to (67.6, 58.5), turned to 0 degrees
- moved R3 6.89 mm to (54.0, 48.3)
- moved MISC-ICON 5.40 mm to (65.9, 55.3)
- moved R4 2.16 mm to (54.3, 53.3)
- moved U2 0.85 mm to (60.0, 50.4)
- moved C3 0.50 mm to (55.7, 44.8)
- moved C4 0.50 mm to (55.7, 46.8)
Connections:
- J3 pad 2: /Prog_TXD -> /ESP32_DM
- J3 pad 3: /Prog_RXD -> /ESP32_DP
- J3 pad 4: /BOOT -> GND
- J3 pad 5: /EN -> Net-(J3-CC1)
- J3 pad 6: GND -> Net-(J3-CC2)
- SW1 pad 2: /SET_SW -> /BOOT
- U2 pad 10: /SET_SW -> unconnected-(U2-IO10-Pad10)
- U2 pad 11: /Prog_TXD -> unconnected-(U2-IO20/RXD-Pad11)
- U2 pad 12: /Prog_RXD -> unconnected-(U2-IO21/TXD-Pad12)
- U2 pad 13: unconnected-(U2-IO18/USB_D--Pad13) -> Net-(U2-IO18/USB_D-)
- U2 pad 14: unconnected-(U2-IO19/USB_D+-Pad14) -> Net-(U2-IO19/USB_D+)
Routing:
- net /EN: track 41.7 -> 3.67 mm
- net /Prog_TXD: track 29.1 -> 0.00 mm, vias 3 -> 0
- net /Prog_RXD: track 27.9 -> 0.00 mm, vias 2 -> 0
- net /SET_SW: track 24.3 -> 0.00 mm, vias 2 -> 0
- net /ESP32_DP: track 0.00 -> 22.1 mm, vias 0 -> 3
- net +3V3: track 49.4 -> 69.4 mm, vias 1 -> 5
- net /ESP32_DM: track 0.00 -> 19.6 mm, vias 0 -> 2
- net Net-(J3-CC1): track 0.00 -> 10.5 mm, vias 0 -> 1
- net VBUS: track 31.3 -> 40.7 mm
- net Net-(J3-CC2): track 0.00 -> 5.36 mm, vias 0 -> 1
- net /BOOT: track 33.7 -> 28.3 mm
- net GND: track 9.67 -> 6.29 mm, vias 68 -> 100
- net /LED: track 17.8 -> 14.8 mm
- net Net-(U2-IO19/USB_D+): track 0.00 -> 2.29 mm, vias 0 -> 1
- net Net-(U2-IO18/USB_D-): track 0.00 -> 2.25 mm, vias 0 -> 1
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Other:
- board size 20 x 41.5 mm -> 20 x 42.4 mm
- board text removed: "5V"
- board text removed: "BT"
- board text removed: "EN"
- board text removed: "GND"
- board text removed: "RXD"
- board text removed: "SET"
- board text removed: "TXD"
