File: 74TH-G071-grove_uart_usb_adapter/74TH-G071-grove_uart_usb_adapter.kicad_pcb (KiCad board)
At the start: 2 copper layers, 14.7 x 32 mm, 17 parts, among them J1 USB2.0-C_SMT, U1 CH340C, U2 CH213K

Commit message: 74TH-G071-grove_uart_usb_adapter/1.1.0
Parts:
- added JP1: Jumper_2_Open, 74th:SolderJumper-2, B.Cu at (79.3, 64.0)
- moved C4 7.03 mm to (83.0, 65.2), turned to -90 degrees
Connections:
- C4 pad 1: +5V -> Net-(CH1-VCC)
- CH1 pad 3: +5V -> Net-(CH1-VCC)
Routing:
- net Net-(CH1-VCC): track 0.00 -> 7.85 mm, vias 0 -> 1
- net +5V: track 26.9 -> 25.3 mm, vias 1 -> 0
- net GND: vias 29 -> 30
Other:
- board text added: "G071-v${REVISION}"
- board text added: "Power Export"
- board text removed: "74TH-G071"
- board text removed: "v1.0.0"
