File: 74TH-G071-grove_uart_usb_adapter/74TH-G071-grove_uart_usb_adapter.kicad_sch (KiCad schematic)
At the start: 15 parts, among them J1 USB2.0-C_SMT, U1 CH340C, U2 CH213K

Commit message: 74TH-G071-grove_uart_usb_adapter/1.1.0
Parts:
- added JP1: Jumper_2_Open, 74th:SolderJumper-2, symbol 74th_Interface:Jumper_2
Connections:
- net +5V: now also JP1.2 (B); no longer C4.1, CH1.3 (VCC)
- new net: C4.1, CH1.3 (VCC), JP1.1 (A)
Other:
- moved on the sheet: C4, CH1, R3, R4, R5, R6
