File: 74TH-G074-M5_Core_port_bottom/74TH-G074-M5_Core_port_bottom.kicad_pcb (KiCad board)
At the start: 2 copper layers, 50 x 50 mm, 11 parts, among them M2 Hole_M2_2.2, M2 Hole_M3_3.2

Commit message: 74TH-G074-M5_Core_port_bottom/1.0.0
Parts:
- moved CH2 2.00 mm to (68.0, 41.0)
- moved CH3 2.00 mm to (86.0, 41.0)
Routing:
- net /GPIO8: track 45.4 -> 47.3 mm
- net /GPIO17: track 49.0 -> 50.7 mm
- net GND: vias 41 -> 49
Other:
- outline, holes or cut-outs redrawn
- board text added: "B"
- board text added: "C"
- board text added: "G0:18 G1:17"
- board text added: "G0:8 G1:9"

Commit message: 74TH-G074-M5_Core_port_bottom/1.0.1
Parts:
- CH1: moved to F.Cu
- CH2, CH3: moved to B.Cu
- moved CH2 2.10 mm to (68.0, 43.1), turned to 0 degrees
- moved CH3 2.10 mm to (86.0, 43.1), turned to 0 degrees
Routing:
- net /GPIO8: track 47.3 -> 8.09 mm
- net /GPIO9: track 36.3 -> 18.3 mm
- net /GPIO18: track 54.6 -> 46.3 mm
- net /GPIO17: track 50.7 -> 45.7 mm
- net GND: vias 49 -> 84
- added copper zone on F.Cu, net +5V
- removed copper zone on B.Cu, net +5V
Other:
- outline, holes or cut-outs redrawn
- board text removed: "${REFERENCE}"
