File: 74TH-G074-M5_Core_port_bottom/74TH-G074-M5_Core_port_bottom.kicad_sch (KiCad schematic)
At the start: 3 parts

Commit message: 74TH-G074-M5_Core_port_bottom/1.0.1
Other:
- title: (none) -> M5 Core Port Bottom
Changed lines of the file:
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@@
 	(generator_version "9.0")
 	(paper "A4")
+	(title_block
+		(title "M5 Core Port Bottom")
+		(rev "1.0.1")
+	)
 	(junction
 		(at 62.23 43.18)
